File: Hardware/Rocket/zenith.brd (EAGLE design)
At the start: 50.9 x 95.3 mm, 167 parts, among them IC1 BD60GC0WEFJ-E2, IC2 BMI088, IC3 BMM150, IC4 BD6211F-E2, IC5 MKL02Z32VFG4, IC6 TPS7A4533KTTR, IC7 MS561101BA03-00, IC9 LE25U40CMC-AH, J1 1727052, J10 142-0701-211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

Commit message: updated ee stuff for the lads on bps discord
Routing:
- net MCU_JTAG_TDI: track 85.5 -> 78.3 mm, vias 1 -> 2
- net N$27: track 27.2 -> 28.1 mm, vias 0 -> 1
- net N$21: track 31.7 -> 32.6 mm
- net N$22: track 29.0 -> 29.8 mm
